Commit message: ✨ feat: add sfm config

File: entities/robots/jackal/urdf/accessories.urdf.xacro (robot description, xacro)
@@ -93,4 +93,5 @@
   </xacro:if>
   <xacro:include filename="$(find arena_simulation_setup)/entities/robots/jackal/urdf/accessories/stereo_camera_mount.urdf.xacro" />
+  <xacro:include filename="$(find pointgrey_camera_description)/urdf/pointgrey_flea3.urdf.xacro" />
   <!-- If enabled, generates a pair of flea3 cameras for stereo vision with a tilt of 30 degrees. -->
   <!-- Disabled temporarily due to metapackage issue. -->

File: entities/robots/jackal/urdf/jackal.urdf.xacro (robot description, xacro)
@@ -229,3 +229,8 @@
   <!-- Optional custom includes. -->
   <xacro:include filename="$(optenv JACKAL_URDF_EXTRAS empty.urdf)" />
+  <xacro:include filename="$(find arena_simulation_setup)/entities/robots/jackal/urdf/accessories/realsense_d415.urdf.xacro"/>
+  <xacro:sensor_d415 name="d415" parent="base_link" use_nominal_extrinsics="true">
+    <!-- <origin xyz="0.061 0.0 0.271" rpy="0 0 0"/> -->
+    <origin xyz="0.061 0.0 1.500" rpy="0 0 0"/>
+  </xacro:sensor_d415>
 </robot>

File: entities/robots/rto/urdf/rto.urdf.xacro (robot description, xacro)
@@ -11,5 +11,6 @@
   </xacro:bracket>
   <xacro:sensor_d415 name="d415" parent="base_link" use_nominal_extrinsics="true">
-    <origin xyz="0.061 0.0 0.271" rpy="0 0 0"/>
+    <!-- <origin xyz="0.061 0.0 0.271" rpy="0 0 0"/> -->
+    <origin xyz="0.061 0.0 1.500" rpy="0 0 0"/>
   </xacro:sensor_d415>
   <xacro:hokuyo name="hokuyo" parent="base_link">

File: entities/robots/rto/urdf/sensors/hokuyo.urdf.xacro (robot description, xacro)
@@ -53,5 +53,5 @@
           </scan>
           <range>
-            <min>0.03</min>
+            <min>0.2</min>
             <max>50</max> <!--5.6-->
             <resolution>0.01</resolution>

File: entities/robots/waffle/urdf/waffle.gazebo.xacro (robot description, xacro)
@@ -1,4 +1,4 @@
 <?xml version="1.0"?>
-<robot name="turtlebot3_waffle_pi_sim" xmlns:xacro="http://ros.org/wiki/xacro">
+<robot name="turtlebot3_waffle_sim" xmlns:xacro="http://ros.org/wiki/xacro">
   <xacro:arg name="laser_visual"  default="false"/>
   <xacro:arg name="camera_visual" default="false"/>
@@ -53,5 +53,5 @@
   </gazebo>
   <gazebo>
-    <plugin name="turtlebot3_waffle_pi_controller" filename="libgazebo_ros_diff_drive.so">
+    <plugin name="turtlebot3_waffle_controller" filename="libgazebo_ros_diff_drive.so">
       <commandTopic>cmd_vel</commandTopic>
       <odometryTopic>odom</odometryTopic>
